File: hardware/137MHz_RF_FrontEnd.kicad_sch (KiCad schematic)
At the start: 39 parts, among them J1 Conn_Coaxial, J2 Conn_Coaxial, J3 Conn_01x02_Pin, Q1 AO3401A, U1 PGA-103

Commit message: Update & applied changes
Parts:
- removed R4, R5: 300, Resistor_SMD:R_0603_1608Metric_Pad0.98x0.95mm_HandSolder, symbol Device:R
- removed R6: 18, Resistor_SMD:R_0603_1608Metric_Pad0.98x0.95mm_HandSolder, symbol Device:R
Connections:
- net at C10.2, C9.1, L11.1: now also C15.1

Commit message: update
Parts:
- L4: value 150nH -> 120nH
Changed lines of the file:
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@@
 			)
 		)
-		(property "Value" "150nH"
+		(property "Value" "120nH"
 			(at 88.9 106.6799 0)
 			(show_name no)

Commit message: update/addedLDO
Parts:
- added C16, C17: 10uF, Capacitor_SMD:C_0805_2012Metric_Pad1.18x1.45mm_HandSolder, symbol Device:C
- added U2: TLV1117-50, Package_TO_SOT_SMD:SOT-223, symbol Regulator_Linear:TLV1117-50
Connections:
- net GND: now also C16.2, C17.2, U2.1 (GND)
- net at FB1.1: now also C17.1, U2.2 (VO); no longer Q1.2 (S)
- new net: C16.1, Q1.2 (S), U2.3 (VI)
Other:
- moved on the sheet: J1, J3
